Commit message: Update fourDOF.urdf

File: src/hw3code/urdf/fourDOF.urdf (robot description, URDF)
Before this commit: robot TestRobot, 6 links, 5 joints
Links:
- removed link frame0prime
- removed link frame1
- removed link frame2
- removed link sphere
- removed link tip
- removed link world
- added link base_link
- added link end_effector; visual box size=0.1 0.1 0.1
- added link link1; visual cylinder length=L radius=0.05
- added link link2; visual cylinder length=L radius=0.05
- added link link3; visual cylinder length=L radius=0.05
- added link link4; visual cylinder length=L radius=0.05
Joints:
- removed joint attach-sphere
- removed joint joint0prime
- removed joint joint2prime
- removed joint theta1
- removed joint theta2
- added joint end_effector_joint: type fixed, parent link4, child end_effector, origin xyz=L 0 0 rpy=0 0 0
- added joint joint1: type continuous, parent base_link, child link1, origin xyz=0 0 0 rpy=0 0 0, axis 0 0 1
- added joint joint2: type continuous, parent link1, child link2, origin xyz=0 0 L rpy=0 0 0, axis 0 1 0
- added joint joint3: type continuous, parent link2, child link3, origin xyz=0 0 L rpy=0 0 0, axis 0 0 1
- added joint joint4: type continuous, parent link3, child link4, origin xyz=0 0 L rpy=0 0 0, axis 0 1 0

Commit message: Update fourDOF.urdf

File: src/hw3code/urdf/fourDOF.urdf (robot description, URDF)
Before this commit: robot FourDOFRobot, 6 links, 5 joints
Links:
- link link1: geometry visual cylinder length=.4 radius=0.05
- link link2: geometry visual cylinder length=.4 radius=0.05
- link link3: geometry visual cylinder length=.4 radius=0.05
- link link4: geometry visual cylinder length=.4 radius=0.05
Joints:
- joint end_effector_joint: origin xyz=L 0 0 rpy=0 0 0 -> xyz=.4 0 0 rpy=0 0 0
- joint joint2: origin xyz=0 0 L rpy=0 0 0 -> xyz=0 0 .4 rpy=0 0 0
- joint joint3: origin xyz=0 0 L rpy=0 0 0 -> xyz=0 0 .4 rpy=0 0 0
- joint joint4: origin xyz=0 0 L rpy=0 0 0 -> xyz=0 0 .4 rpy=0 0 0

Commit message: Update fourDOF.urdf

File: src/hw3code/urdf/fourDOF.urdf (robot description, URDF)
Before this commit: robot FourDOFRobot, 6 links, 5 joints
Links:
- removed link base_link
- removed link end_effector
- removed link link1
- removed link link2
- removed link link3
- removed link link4
- added link frame0prime
- added link frame1
- added link frame2
- added link frame3
- added link frame4
- added link tip
- added link world
Joints:
- removed joint end_effector_joint
- removed joint joint1
- removed joint joint2
- removed joint joint3
- removed joint joint4
- added joint shift0: type fixed, parent world, child frame0prime, origin xyz=0 0 0.2 rpy=0 0 0
- added joint shift4: type fixed, parent frame4, child tip, origin xyz=0 0 -0.2 rpy=0 0 0
- added joint theta1: type continuous, parent frame0prime, child frame1, axis 0 0 1
- added joint theta2: type continuous, parent frame1, child frame2, origin xyz=0.2 0 0.2 rpy=0 0 0, axis 1 0 0
- added joint theta3: type continuous, parent frame2, child frame3, origin xyz=0.2 -0.2 0 rpy=0 0 0, axis 0 1 0
- added joint theta4: type continuous, parent frame3, child frame4, origin xyz=0 0.2 -0.2 rpy=0 0 0, axis 0 0 1

Commit message: Update fourDOF.urdf

File: src/hw3code/urdf/fourDOF.urdf (robot description, URDF)
Before this commit: robot FourDOF, 7 links, 6 joints
Links:
- removed link frame0prime
- removed link tip
- added link frame1prime
- added link frame2prime
- added link frame3prime
- added link frameTip
Joints:
- removed joint shift4
- added joint shift1prime: type fixed, parent frame1prime, child frame2, origin xyz=0 0.2 0 rpy=0 0 0
- added joint shift2prime: type fixed, parent frame2prime, child frame3, origin xyz=0 0 -0.2 rpy=0 0 0
- added joint shift3prime: type fixed, parent frame3prime, child frame4, origin xyz=0 0.2 0 rpy=0 0 0
- joint shift0: child frame0prime -> frame1
- joint theta1: child frame1 -> frame1prime; origin (none) -> xyz=0 0 0.2 rpy=0 0 0; parent frame0prime -> frame1
- joint theta2: axis 1 0 0 -> 0 1 0; child frame2 -> frame2prime; origin xyz=0.2 0 0.2 rpy=0 0 0 -> xyz=0 0.2 0 rpy=0 0 0; parent frame1 -> frame2
- joint theta3: axis 0 1 0 -> 0 0 -1; child frame3 -> frame3prime; origin xyz=0.2 -0.2 0 rpy=0 0 0 -> xyz=0 0 -0.2 rpy=0 0 0; parent frame2 -> frame3
- joint theta4: axis 0 0 1 -> 0 1 0; child frame4 -> frameTip; origin xyz=0 0.2 -0.2 rpy=0 0 0 -> xyz=0 0.2 0 rpy=0 0 0; parent frame3 -> frame4
